File: hardware/cm4-digipi-carrier/cm4-digipi-carrier.kicad_pcb (KiCad board)
At the start: 2 copper layers, 40 x 55 mm, 1 part

Commit message: Initial Commit.
Parts:
- added C1: 220uF, my_components:Cap_Elec_Radial_6.3mm, F.Cu at (213.9, 55.9)
- added C12: 22pF, Capacitor_SMD:C_0603_1608Metric_Pad1.08x0.95mm_HandSolder, F.Cu at (239.4, 48.0)
- added C13: 22pF, Capacitor_SMD:C_0603_1608Metric_Pad1.08x0.95mm_HandSolder, F.Cu at (193.9, 74.7)
- added C14: 1uF, my_components:Cap_Elec_Radial_5mm, F.Cu at (253.0, 31.1)
- added C15: 1uF, my_components:Cap_Elec_Radial_5mm, F.Cu at (226.8, 54.7)
- added C2: 220uF, my_components:Cap_Elec_Radial_6.3mm, F.Cu at (227.4, 48.0)
- added C3: 10uF, my_components:Cap_Elec_Radial_5mm, F.Cu at (253.0, 37.2)
- added C4: 10uF, my_components:Cap_Elec_Radial_5mm, F.Cu at (234.2, 47.3)
- added CR1: SMBJ5.0A-TR, SMBJ5.0A-TR:SMBJ5.0A-TR, F.Cu at (177.8, 118.4)
- added D1: LED Green, LED_SMD:LED_0603_1608Metric, F.Cu at (184.9, 127.0)
- added D2: LED Red, LED_SMD:LED_0603_1608Metric, F.Cu at (184.9, 124.5)
- added D3: RX LED, LED_SMD:LED_0603_1608Metric, F.Cu at (178.1, 80.3)
- added D4: PTT LED, LED_SMD:LED_0603_1608Metric, F.Cu at (172.2, 80.3)
- added J1: USB4105-GF-A, USB4105-GF-A:GCT_USB4105-GF-A, F.Cu at (173.4, 130.9)
- added J2: 6P6C, ul_SS-90000-003:SS-90000-003, F.Cu at (122.6, 95.5)
- added JP1: ID_WP, my_components:Conn_Pin_Header_2x1_2.54mm_NoKey, F.Cu at (220.7, 53.5)
- added MOSFET1: PTT Fet, ul_RHU002N06FRAT106:RHU002N06FRAT106, F.Cu at (172.2, 89.9)
- added P1: Headphones, my_components:Conn_Audio_3.5mm_Stereo_SJ1-353XNG, F.Cu at (106.8, 123.7)
- added P2: Line Output, my_components:Conn_Audio_3.5mm_Stereo, F.Cu at (106.7, 113.3)
- added P4: Line Input, my_components:Conn_Audio_3.5mm_Stereo, F.Cu at (119.9, 28.0)
- added R1: 100, Resistor_SMD:R_0603_1608Metric_Pad0.98x0.95mm_HandSolder, F.Cu at (262.5, 31.8)
- added R10: 33, Resistor_SMD:R_0603_1608Metric_Pad0.98x0.95mm_HandSolder, F.Cu at (218.3, 49.9)
- added R11: 1k, Resistor_SMD:R_0603_1608Metric_Pad0.98x0.95mm_HandSolder, F.Cu at (262.5, 29.3)
- added R12: 3.9k, Resistor_SMD:R_0603_1608Metric_Pad0.98x0.95mm_HandSolder, F.Cu at (258.2, 34.3)
- added R13: 3.9k, Resistor_SMD:R_0603_1608Metric_Pad0.98x0.95mm_HandSolder, F.Cu at (233.3, 51.6)
- added R14: 33, Resistor_SMD:R_0603_1608Metric_Pad0.98x0.95mm_HandSolder, F.Cu at (232.1, 56.7)
- added R15: 33, Resistor_SMD:R_0603_1608Metric_Pad0.98x0.95mm_HandSolder, F.Cu at (236.4, 56.7)
- added R16: 5.1k, Resistor_SMD:R_0603_1608Metric_Pad0.98x0.95mm_HandSolder, F.Cu at (170.2, 123.4)
- added R17: 5.6k, Resistor_SMD:R_0603_1608Metric_Pad0.98x0.95mm_HandSolder, F.Cu at (258.2, 31.8)
- added R18: 5.6k, Resistor_SMD:R_0603_1608Metric_Pad0.98x0.95mm_HandSolder, F.Cu at (243.8, 50.5)
- added R19: 1k, Resistor_SMD:R_0603_1608Metric_Pad0.98x0.95mm_HandSolder, F.Cu at (180.8, 127.0)
- added R2: 100, Resistor_SMD:R_0603_1608Metric_Pad0.98x0.95mm_HandSolder, F.Cu at (243.8, 48.0)
- added R20: 5.6k, Resistor_SMD:R_0603_1608Metric_Pad0.98x0.95mm_HandSolder, F.Cu at (252.1, 41.5)
- added R21: 5.6k, Resistor_SMD:R_0603_1608Metric_Pad0.98x0.95mm_HandSolder, F.Cu at (243.8, 45.5)
- added R22: 5.1k, Resistor_SMD:R_0603_1608Metric_Pad0.98x0.95mm_HandSolder, F.Cu at (174.2, 123.4)
- added R23: 1k, Resistor_SMD:R_0603_1608Metric_Pad0.98x0.95mm_HandSolder, F.Cu at (169.7, 117.9)
- added R24: 200, ul_ERJ3EKF2000V:ERJ3EKF2000V, F.Cu at (177.8, 84.8)
- added R25: 100k, Resistor_SMD:R_0603_1608Metric_Pad0.98x0.95mm_HandSolder, F.Cu at (172.2, 84.8)
- added R26: 200, ul_ERJ3EKF2000V:ERJ3EKF2000V, F.Cu at (240.8, 98.0)
- added R3: 47k, Resistor_SMD:R_0603_1608Metric_Pad0.98x0.95mm_HandSolder, F.Cu at (239.4, 50.5)
- added R4: 47k, Resistor_SMD:R_0603_1608Metric_Pad0.98x0.95mm_HandSolder, F.Cu at (258.2, 29.3)
- added R5: 47k, Resistor_SMD:R_0603_1608Metric_Pad0.98x0.95mm_HandSolder, F.Cu at (252.1, 44.0)
- added R6: 47k, Resistor_SMD:R_0603_1608Metric_Pad0.98x0.95mm_HandSolder, F.Cu at (236.4, 54.1)
- added R7: 33, Resistor_SMD:R_0603_1608Metric_Pad0.98x0.95mm_HandSolder, F.Cu at (239.4, 45.5)
- added R8: 33, Resistor_SMD:R_0603_1608Metric_Pad0.98x0.95mm_HandSolder, F.Cu at (258.2, 36.8)
- added R9: 33, Resistor_SMD:R_0603_1608Metric_Pad0.98x0.95mm_HandSolder, F.Cu at (232.1, 54.1)
- added U1: 24LC32, my_components:IC_SOIC8_Narrow, F.Cu at (213.2, 48.2)
- added U2: TPS79333DBVR, my_components:IC_SOT23-5_Hand_Soldering, F.Cu at (220.5, 57.7)
- added U3: WM8731CLSEFL, Package_DFN_QFN:QFN-28-1EP_5x5mm_P0.5mm_EP3.35x3.35mm, F.Cu at (147.3, 85.9)
- added U4: 74LVC1G07SE-7, Package_TO_SOT_SMD:SOT-353_SC-70-5, F.Cu at (169.7, 113.3)
- added X1: 12.288MHz, my_components:Crystal_5.0x3.2mm, F.Cu at (219.9, 46.4)
- moved Module1 1.34 mm to (164.3, 81.8)
Connections:
- net Net-(Module1-Pad57) renamed SD_CLK
- Module1 pad 1: Net-(Module1-Pad1) -> GND
- Module1 pad 10: Net-(Module1-Pad10) -> unconnected-(Module1-Pad10)
- Module1 pad 100: Net-(Module1-Pad100) -> unconnected-(Module1-Pad100)
- Module1 pad 101: Net-(Module1-Pad101) -> unconnected-(Module1-Pad101)
- Module1 pad 102: Net-(Module1-Pad102) -> unconnected-(Module1-Pad102)
- Module1 pad 103: Net-(Module1-Pad103) -> unconnected-(Module1-Pad103)
- Module1 pad 104: Net-(Module1-Pad104) -> unconnected-(Module1-Pad104)
- Module1 pad 105: Net-(Module1-Pad105) -> unconnected-(Module1-Pad105)
- Module1 pad 106: Net-(Module1-Pad106) -> unconnected-(Module1-Pad106)
- Module1 pad 107: Net-(Module1-Pad107) -> GND
- Module1 pad 108: Net-(Module1-Pad108) -> GND
- Module1 pad 109: Net-(Module1-Pad109) -> unconnected-(Module1-Pad109)
- Module1 pad 11: Net-(Module1-Pad11) -> unconnected-(Module1-Pad11)
- Module1 pad 110: Net-(Module1-Pad110) -> unconnected-(Module1-Pad110)
- Module1 pad 111: Net-(Module1-Pad111) -> unconnected-(Module1-Pad111)
- Module1 pad 112: Net-(Module1-Pad112) -> unconnected-(Module1-Pad112)
- Module1 pad 113: Net-(Module1-Pad113) -> GND
- Module1 pad 114: Net-(Module1-Pad114) -> GND
- Module1 pad 115: Net-(Module1-Pad115) -> unconnected-(Module1-Pad115)
- Module1 pad 116: Net-(Module1-Pad116) -> unconnected-(Module1-Pad116)
- Module1 pad 117: Net-(Module1-Pad117) -> unconnected-(Module1-Pad117)
- Module1 pad 118: Net-(Module1-Pad118) -> unconnected-(Module1-Pad118)
- Module1 pad 119: Net-(Module1-Pad119) -> GND
- Module1 pad 12: Net-(Module1-Pad12) -> unconnected-(Module1-Pad12)
- Module1 pad 120: Net-(Module1-Pad120) -> GND
- Module1 pad 121: Net-(Module1-Pad121) -> unconnected-(Module1-Pad121)
- Module1 pad 122: Net-(Module1-Pad122) -> unconnected-(Module1-Pad122)
- Module1 pad 123: Net-(Module1-Pad123) -> unconnected-(Module1-Pad123)
- Module1 pad 124: Net-(Module1-Pad124) -> unconnected-(Module1-Pad124)
- Module1 pad 125: Net-(Module1-Pad125) -> GND
- Module1 pad 126: Net-(Module1-Pad126) -> GND
- Module1 pad 127: Net-(Module1-Pad127) -> unconnected-(Module1-Pad127)
- Module1 pad 128: Net-(Module1-Pad128) -> unconnected-(Module1-Pad128)
- Module1 pad 129: Net-(Module1-Pad129) -> unconnected-(Module1-Pad129)
- Module1 pad 13: Net-(Module1-Pad13) -> GND
- Module1 pad 130: Net-(Module1-Pad130) -> unconnected-(Module1-Pad130)
- Module1 pad 131: Net-(Module1-Pad131) -> GND
- Module1 pad 132: Net-(Module1-Pad132) -> GND
- Module1 pad 133: Net-(Module1-Pad133) -> unconnected-(Module1-Pad133)
- Module1 pad 134: Net-(Module1-Pad134) -> unconnected-(Module1-Pad134)
- Module1 pad 135: Net-(Module1-Pad135) -> unconnected-(Module1-Pad135)
- Module1 pad 136: Net-(Module1-Pad136) -> unconnected-(Module1-Pad136)
- Module1 pad 137: Net-(Module1-Pad137) -> GND
- Module1 pad 138: Net-(Module1-Pad138) -> GND
- Module1 pad 139: Net-(Module1-Pad139) -> unconnected-(Module1-Pad139)
- Module1 pad 14: Net-(Module1-Pad14) -> GND
- Module1 pad 140: Net-(Module1-Pad140) -> unconnected-(Module1-Pad140)
- Module1 pad 141: Net-(Module1-Pad141) -> unconnected-(Module1-Pad141)
- Module1 pad 142: Net-(Module1-Pad142) -> unconnected-(Module1-Pad142)
- Module1 pad 143: Net-(Module1-Pad143) -> unconnected-(Module1-Pad143)
- Module1 pad 144: Net-(Module1-Pad144) -> GND
- Module1 pad 145: Net-(Module1-Pad145) -> unconnected-(Module1-Pad145)
- Module1 pad 146: Net-(Module1-Pad146) -> unconnected-(Module1-Pad146)
- Module1 pad 147: Net-(Module1-Pad147) -> unconnected-(Module1-Pad147)
- Module1 pad 148: Net-(Module1-Pad148) -> unconnected-(Module1-Pad148)
- Module1 pad 149: Net-(Module1-Pad149) -> unconnected-(Module1-Pad149)
- Module1 pad 15: Net-(Module1-Pad15) -> unconnected-(Module1-Pad15)
- Module1 pad 150: Net-(Module1-Pad150) -> GND
- Module1 pad 151: Net-(Module1-Pad151) -> unconnected-(Module1-Pad151)
- Module1 pad 152: Net-(Module1-Pad152) -> unconnected-(Module1-Pad152)
- Module1 pad 153: Net-(Module1-Pad153) -> unconnected-(Module1-Pad153)
- Module1 pad 154: Net-(Module1-Pad154) -> unconnected-(Module1-Pad154)
- Module1 pad 155: Net-(Module1-Pad155) -> GND
- Module1 pad 156: Net-(Module1-Pad156) -> GND
- Module1 pad 157: Net-(Module1-Pad157) -> unconnected-(Module1-Pad157)
- Module1 pad 158: Net-(Module1-Pad158) -> unconnected-(Module1-Pad158)
- Module1 pad 159: Net-(Module1-Pad159) -> unconnected-(Module1-Pad159)
- Module1 pad 16: Net-(Module1-Pad16) -> unconnected-(Module1-Pad16)
- Module1 pad 160: Net-(Module1-Pad160) -> unconnected-(Module1-Pad160)
- Module1 pad 161: Net-(Module1-Pad161) -> GND
- Module1 pad 162: Net-(Module1-Pad162) -> GND
- Module1 pad 163: Net-(Module1-Pad163) -> unconnected-(Module1-Pad163)
- Module1 pad 164: Net-(Module1-Pad164) -> unconnected-(Module1-Pad164)
- Module1 pad 165: Net-(Module1-Pad165) -> unconnected-(Module1-Pad165)
- Module1 pad 166: Net-(Module1-Pad166) -> unconnected-(Module1-Pad166)
- Module1 pad 167: Net-(Module1-Pad167) -> GND
- Module1 pad 168: Net-(Module1-Pad168) -> GND
- Module1 pad 169: Net-(Module1-Pad169) -> unconnected-(Module1-Pad169)
- Module1 pad 17: Net-(Module1-Pad17) -> unconnected-(Module1-Pad17)
- Module1 pad 170: Net-(Module1-Pad170) -> unconnected-(Module1-Pad170)
- Module1 pad 171: Net-(Module1-Pad171) -> unconnected-(Module1-Pad171)
- Module1 pad 172: Net-(Module1-Pad172) -> unconnected-(Module1-Pad172)
- Module1 pad 173: Net-(Module1-Pad173) -> GND
- Module1 pad 174: Net-(Module1-Pad174) -> GND
- Module1 pad 175: Net-(Module1-Pad175) -> unconnected-(Module1-Pad175)
- Module1 pad 176: Net-(Module1-Pad176) -> unconnected-(Module1-Pad176)
- Module1 pad 177: Net-(Module1-Pad177) -> unconnected-(Module1-Pad177)
- Module1 pad 178: Net-(Module1-Pad178) -> unconnected-(Module1-Pad178)
- Module1 pad 179: Net-(Module1-Pad179) -> GND
- Module1 pad 18: Net-(Module1-Pad18) -> unconnected-(Module1-Pad18)
- Module1 pad 180: Net-(Module1-Pad180) -> GND
- Module1 pad 181: Net-(Module1-Pad181) -> unconnected-(Module1-Pad181)
- Module1 pad 182: Net-(Module1-Pad182) -> unconnected-(Module1-Pad182)
- Module1 pad 183: Net-(Module1-Pad183) -> unconnected-(Module1-Pad183)
- Module1 pad 184: Net-(Module1-Pad184) -> unconnected-(Module1-Pad184)
- Module1 pad 185: Net-(Module1-Pad185) -> GND
- Module1 pad 186: Net-(Module1-Pad186) -> GND
- Module1 pad 187: Net-(Module1-Pad187) -> unconnected-(Module1-Pad187)
- Module1 pad 188: Net-(Module1-Pad188) -> unconnected-(Module1-Pad188)
- Module1 pad 189: Net-(Module1-Pad189) -> unconnected-(Module1-Pad189)
- Module1 pad 19: Net-(Module1-Pad19) -> unconnected-(Module1-Pad19)
- Module1 pad 190: Net-(Module1-Pad190) -> unconnected-(Module1-Pad190)
- Module1 pad 191: Net-(Module1-Pad191) -> GND
- Module1 pad 192: Net-(Module1-Pad192) -> GND
- Module1 pad 193: Net-(Module1-Pad193) -> unconnected-(Module1-Pad193)
- Module1 pad 194: Net-(Module1-Pad194) -> unconnected-(Module1-Pad194)
- Module1 pad 195: Net-(Module1-Pad195) -> unconnected-(Module1-Pad195)
- Module1 pad 196: Net-(Module1-Pad196) -> unconnected-(Module1-Pad196)
- Module1 pad 197: Net-(Module1-Pad197) -> GND
- Module1 pad 198: Net-(Module1-Pad198) -> GND
- Module1 pad 199: Net-(Module1-Pad199) -> unconnected-(Module1-Pad199)
- Module1 pad 2: Net-(Module1-Pad2) -> GND
- Module1 pad 20: Net-(Module1-Pad20) -> unconnected-(Module1-Pad20)
- Module1 pad 200: Net-(Module1-Pad200) -> unconnected-(Module1-Pad200)
- Module1 pad 21: Net-(Module1-Pad21) -> /CM4 GPIO/nLED_Activity
- Module1 pad 22: Net-(Module1-Pad22) -> GND
- Module1 pad 23: Net-(Module1-Pad23) -> GND
- Module1 pad 24: Net-(Module1-Pad24) -> GPIO26
- Module1 pad 25: Net-(Module1-Pad25) -> GPIO21/PCM_DOUT
- Module1 pad 26: Net-(Module1-Pad26) -> GPIO19/PCM_FS
- Module1 pad 27: Net-(Module1-Pad27) -> GPIO20/PCM_DIN
- Module1 pad 28: Net-(Module1-Pad28) -> unconnected-(Module1-Pad28)
- Module1 pad 29: Net-(Module1-Pad29) -> GPIO16
- Module1 pad 3: Net-(Module1-Pad3) -> unconnected-(Module1-Pad3)
- Module1 pad 30: Net-(Module1-Pad30) -> unconnected-(Module1-Pad30)
- Module1 pad 31: Net-(Module1-Pad31) -> GPIO12
- Module1 pad 32: Net-(Module1-Pad32) -> GND
- Module1 pad 33: Net-(Module1-Pad33) -> GND
- Module1 pad 34: Net-(Module1-Pad34) -> unconnected-(Module1-Pad34)
- Module1 pad 35: Net-(Module1-Pad35) -> ID_SC
- Module1 pad 36: Net-(Module1-Pad36) -> ID_SD
- Module1 pad 37: Net-(Module1-Pad37) -> unconnected-(Module1-Pad37)
- Module1 pad 38: Net-(Module1-Pad38) -> unconnected-(Module1-Pad38)
- Module1 pad 39: Net-(Module1-Pad39) -> unconnected-(Module1-Pad39)
- Module1 pad 4: Net-(Module1-Pad4) -> unconnected-(Module1-Pad4)
- Module1 pad 40: Net-(Module1-Pad40) -> unconnected-(Module1-Pad40)
- Module1 pad 41: Net-(Module1-Pad41) -> unconnected-(Module1-Pad41)
- Module1 pad 42: Net-(Module1-Pad42) -> GND
- Module1 pad 43: Net-(Module1-Pad43) -> GND
- Module1 pad 44: Net-(Module1-Pad44) -> unconnected-(Module1-Pad44)
- Module1 pad 45: Net-(Module1-Pad45) -> unconnected-(Module1-Pad45)
- Module1 pad 46: Net-(Module1-Pad46) -> unconnected-(Module1-Pad46)
- Module1 pad 47: Net-(Module1-Pad47) -> unconnected-(Module1-Pad47)
- Module1 pad 48: Net-(Module1-Pad48) -> unconnected-(Module1-Pad48)
- Module1 pad 49: Net-(Module1-Pad49) -> GPIO18/PCM_CLK
- Module1 pad 5: Net-(Module1-Pad5) -> unconnected-(Module1-Pad5)
- Module1 pad 50: Net-(Module1-Pad50) -> unconnected-(Module1-Pad50)
- Module1 pad 51: Net-(Module1-Pad51) -> unconnected-(Module1-Pad51)
- Module1 pad 52: Net-(Module1-Pad52) -> GND
- Module1 pad 53: Net-(Module1-Pad53) -> GND
- Module1 pad 54: Net-(Module1-Pad54) -> unconnected-(Module1-Pad54)
- Module1 pad 55: Net-(Module1-Pad55) -> unconnected-(Module1-Pad55)
- Module1 pad 56: Net-(Module1-Pad56) -> unconnected-(Module1-Pad56)
- Module1 pad 58: Net-(Module1-Pad58) -> unconnected-(Module1-Pad58)
- Module1 pad 59: Net-(Module1-Pad59) -> GND
- Module1 pad 6: Net-(Module1-Pad6) -> unconnected-(Module1-Pad6)
- Module1 pad 60: Net-(Module1-Pad60) -> GND
- Module1 pad 61: Net-(Module1-Pad61) -> unconnected-(Module1-Pad61)
- Module1 pad 62: Net-(Module1-Pad62) -> unconnected-(Module1-Pad62)
- Module1 pad 63: Net-(Module1-Pad63) -> unconnected-(Module1-Pad63)
- Module1 pad 64: Net-(Module1-Pad64) -> unconnected-(Module1-Pad64)
- Module1 pad 65: Net-(Module1-Pad65) -> GND
- Module1 pad 66: Net-(Module1-Pad66) -> GND
- Module1 pad 67: Net-(Module1-Pad67) -> unconnected-(Module1-Pad67)
- Module1 pad 68: Net-(Module1-Pad68) -> unconnected-(Module1-Pad68)
- Module1 pad 69: Net-(Module1-Pad69) -> unconnected-(Module1-Pad69)
- Module1 pad 7: Net-(Module1-Pad7) -> GND
- Module1 pad 70: Net-(Module1-Pad70) -> unconnected-(Module1-Pad70)
- Module1 pad 71: Net-(Module1-Pad71) -> GND
- Module1 pad 72: Net-(Module1-Pad72) -> unconnected-(Module1-Pad72)
- Module1 pad 73: Net-(Module1-Pad73) -> unconnected-(Module1-Pad73)
- Module1 pad 74: Net-(Module1-Pad74) -> GND
- Module1 pad 75: Net-(Module1-Pad75) -> unconnected-(Module1-Pad75)
- Module1 pad 76: Net-(Module1-Pad76) -> unconnected-(Module1-Pad76)
- Module1 pad 77: Net-(Module1-Pad77) -> +5V
- Module1 pad 78: Net-(Module1-Pad78) -> unconnected-(Module1-Pad78)
- Module1 pad 79: Net-(Module1-Pad79) -> +5V
- Module1 pad 8: Net-(Module1-Pad8) -> GND
- Module1 pad 80: Net-(Module1-Pad80) -> SCL
- Module1 pad 81: Net-(Module1-Pad81) -> +5V
- Module1 pad 82: Net-(Module1-Pad82) -> SDA
- Module1 pad 83: Net-(Module1-Pad83) -> +5V
- Module1 pad 84: Net-(Module1-Pad84) -> +3.3V
- Module1 pad 85: Net-(Module1-Pad85) -> +5V
- Module1 pad 86: Net-(Module1-Pad86) -> +3.3V
- Module1 pad 87: Net-(Module1-Pad87) -> +5V
- Module1 pad 88: Net-(Module1-Pad88) -> +1.8V
- Module1 pad 89: Net-(Module1-Pad89) -> unconnected-(Module1-Pad89)
- Module1 pad 9: Net-(Module1-Pad9) -> unconnected-(Module1-Pad9)
- Module1 pad 90: Net-(Module1-Pad90) -> +1.8V
- Module1 pad 91: Net-(Module1-Pad91) -> unconnected-(Module1-Pad91)
- Module1 pad 92: Net-(Module1-Pad92) -> unconnected-(Module1-Pad92)
- Module1 pad 93: Net-(Module1-Pad93) -> unconnected-(Module1-Pad93)
- Module1 pad 94: Net-(Module1-Pad94) -> unconnected-(Module1-Pad94)
- Module1 pad 95: Net-(Module1-Pad95) -> /CM4 GPIO/nPWR_LED
- Module1 pad 96: Net-(Module1-Pad96) -> unconnected-(Module1-Pad96)
- Module1 pad 97: Net-(Module1-Pad97) -> unconnected-(Module1-Pad97)
- Module1 pad 98: Net-(Module1-Pad98) -> GND
- Module1 pad 99: Net-(Module1-Pad99) -> unconnected-(Module1-Pad99)
Other:
- board size 40 x 55 mm -> 81.8 x 55.4 mm
