File: hardware/cm4-digipi-carrier/cm4-digipi-carrier.kicad_sch (KiCad schematic)
At the start: 0 parts

Commit message: Initial Commit.
Other:
- added sheet Audio Component (audio.kicad_sch)
- added sheet HAM PTT Control (ham_ptt.kicad_sch)
- title: Raspberry Pi Compute Module 4 Carrier Template -> Raspberry Pi Compute Module 4 Digipi Carrier Board
