File: hardware/cm4-digipi-carrier/cm4-gpio.kicad_sch (KiCad schematic)
At the start: 1 part

Commit message: Initial Commit.
Parts:
- added CR1: SMBJ5.0A-TR, SMBJ5.0A-TR:SMBJ5.0A-TR, symbol 2020-11-06_22-01-36:SMBJ5.0A-TR
- added D1: LED Green, LED_SMD:LED_0603_1608Metric, symbol Device:LED
- added D2: LED Red, LED_SMD:LED_0603_1608Metric, symbol Device:LED
- added J1: USB4105-GF-A, USB4105-GF-A:GCT_USB4105-GF-A, symbol USB4105-GF-A:USB4105-GF-A
- added R16, R22: 5.1k, Resistor_SMD:R_0603_1608Metric_Pad0.98x0.95mm_HandSolder, symbol Device:R
- added R19, R23: 1k, Resistor_SMD:R_0603_1608Metric_Pad0.98x0.95mm_HandSolder, symbol Device:R
- added U4: 74LVC1G07SE-7, Package_TO_SOT_SMD:SOT-353_SC-70-5, symbol CM4IO:74LVC1G07_copy
Connections:
- net +3.3V: now also D1.2 (A), D2.2 (A), U4.5 (VCC)
- net +5V: now also CR1.1, J1.A4/B9 (VBUS), J1.B4/A9 (VBUS)
- net GND: now also CR1.2, J1.A1/B12 (GND), J1.B1/A12 (GND), J1.G1 (GND), J1.G2 (GND), J1.G3 (GND), J1.G4 (GND), R16.2, R22.2, U4.3 (GND)
- net nLED_Activity: now reaches Module1.21 (PI_nLED_Activity)
- net nLED_Activity: now also R19.2
- net GPIO26: now reaches Module1.24 (GPIO26)
- net GPIO21/PCM_DOUT: now reaches Module1.25 (GPIO21)
- net GPIO19/PCM_FS: now reaches Module1.26 (GPIO19)
- net GPIO20/PCM_DIN: now reaches Module1.27 (GPIO20)
- net GPIO16: now reaches Module1.29 (GPIO16)
- net GPIO12: now reaches Module1.31 (GPIO12)
- net ID_SC: now reaches Module1.35 (ID_SC)
- net ID_SD: now reaches Module1.36 (ID_SD)
- net GPIO18/PCM_CLK: now reaches Module1.49 (GPIO18)
- net SD_CLK: now reaches Module1.57 (SD_CLK)
- net SCL: now reaches Module1.80 (SCL0)
- net SDA: now reaches Module1.82 (SDA0)
- net nPWR_LED: now reaches Module1.95 (nPI_LED_PWR)
- net nPWR_LED: now also U4.2
- new net: J1.A5 (CC1), R16.1
- new net: J1.B5 (CC2), R22.1
- new net: D2.1 (K), R23.1
- new net: R23.2, U4.4
- new net: D1.1 (K), R19.1
- no-connect marks 0 -> 62
Other:
- note added: "Activity LED"
- note added: "PWR LED"
- note added: "USB-C (Power Only)"
- title: Raspberry Pi Compute Module 4 Carrier Template -> Raspberry Pi Compute Module 4 Digipi Carrier Board
