File: hardware/cm4-digipi-carrier/cm4-high-speed.kicad_sch (KiCad schematic)
At the start: 1 part

Commit message: Initial Commit.
Connections:
- no-connect marks 0 -> 71
Other:
- title: Raspberry Pi Compute Module 4 Carrier Template -> Raspberry Pi Compute Module 4 Digipi Carrier Board
